File: PCB/CONNECTORS.sch (KiCad schematic (older format))
At the start: 11 parts, among them J1 Conn_Coaxial, J2 Conn_ARM_JTAG_SWD_10, J3 67068-8000, J4 PLR135/T9, J5 Conn_02x07_Odd_Even, J6 Conn_01x03, U3 NBA3N012C

Commit message: First fully routed version
Parts:
- J5: value Conn_02x07_Odd_Even -> Conn_02x08_Odd_Even; footprint Connector_PinHeader_2.54mm:PinHeader_2x07_P2.54mm_Vertical -> Connector_PinHeader_2.54mm:PinHeader_2x08_P2.54mm_Vertical; symbol Connector_Generic:Conn_02x07_Odd_Even -> Connector_Generic:Conn_02x08_Odd_Even
Connections:
- net GND: now also J5.15 (Pin_15), J5.16 (Pin_16); no longer J5.13 (Pin_13), J5.14 (Pin_14)
- net VDD3V3: now also J5.13 (Pin_13), J5.14 (Pin_14)
- net RST1 renamed RESET1
- net RST2 renamed RESET2
Changed lines of the file:
@@
 L power:GND #PWR020
 U 1 1 5C37BE12
-P 8000 4100
-F 0 "#PWR020" H 8000 3850 50  0001 C CNN
-F 1 "GND" V 8005 3972 50  0000 R CNN
-F 2 "" H 8000 4100 50  0001 C CNN
-F 3 "" H 8000 4100 50  0001 C CNN
-	1    8000 4100
+P 8000 4200
+F 0 "#PWR020" H 8000 3950 50  0001 C CNN
+F 1 "GND" V 8005 4072 50  0000 R CNN
+F 2 "" H 8000 4200 50  0001 C CNN
+F 3 "" H 8000 4200 50  0001 C CNN
+	1    8000 4200
 	0    -1   -1   0
 $EndComp
@@
 L power:GND #PWR018
 U 1 1 5C37BE88
-P 7500 4100
-F 0 "#PWR018" H 7500 3850 50  0001 C CNN
-F 1 "GND" V 7505 3972 50  0000 R CNN
-F 2 "" H 7500 4100 50  0001 C CNN
-F 3 "" H 7500 4100 50  0001 C CNN
-	1    7500 4100
+P 7500 4200
+F 0 "#PWR018" H 7500 3950 50  0001 C CNN
+F 1 "GND" V 7505 4072 50  0000 R CNN
+F 2 "" H 7500 4200 50  0001 C CNN
+F 3 "" H 7500 4200 50  0001 C CNN
+	1    7500 4200
 	0    1    1    0
 $EndComp
@@
 I2S_MCLK_2
 $Comp
-L Connector_Generic:Conn_02x07_Odd_Even J5
+L Connector_Generic:Conn_02x08_Odd_Even J5
 U 1 1 5C37E504
 P 7700 3800
 F 0 "J5" H 7750 4317 50  0000 C CNN
-F 1 "Conn_02x07_Odd_Even" H 7750 4226 50  0000 C CNN
-F 2 "Connector_PinHeader_2.54mm:PinHeader_2x07_P2.54mm_Vertical" H 7700 3800 50  0001 C CNN
+F 1 "Conn_02x08_Odd_Even" H 7750 4226 50  0000 C CNN
+F 2 "Connector_PinHeader_2.54mm:PinHeader_2x08_P2.54mm_Vertical" H 7700 3800 50  0001 C CNN
 F 3 "~" H 7700 3800 50  0001 C CNN
 	1    7700 3800
@@
 $EndComp
 Text HLabel 7500 3900 0    50   Input ~ 0
-RST1
+RESET1
 Text HLabel 8000 3900 2    50   Input ~ 0
-RST2
+RESET2
 Text HLabel 8000 4000 2    50   Input ~ 0
 I2C_SDA
@@
 Text HLabel 5000 6700 2    50   Input ~ 0
 SPDIF_COAXIAL
+Text HLabel 7500 4100 0    50   Input ~ 0
+VDD3V3
+Text HLabel 8000 4100 2    50   Input ~ 0
+VDD3V3
 $EndSCHEMATC
