File: PCB/STM32F7.sch (KiCad schematic (older format))
At the start: 23 parts, among them U1 STM32F765NIHx

Commit message: First fully routed version
Connections:
- net CRESET: now reaches U1.A1 (PE4)
- net CDONE: now reaches U1.B1 (PE5)
- net RESET1: now reaches U1.R6 (PJ0)
- net RESET2: now reaches U1.R7 (PJ1)
Changed lines of the file:
@@
 Text HLabel 7200 2900 2    50   Input ~ 0
 SS
+Text HLabel 3900 5200 0    50   Input ~ 0
+CRESET
+Text HLabel 3900 5100 0    50   Input ~ 0
+CDONE
+Text HLabel 7200 9000 2    50   Input ~ 0
+RESET1
+Text HLabel 7200 8900 2    50   Input ~ 0
+RESET2
 $EndSCHEMATC
