File: PCB/yui.kicad_pcb (KiCad board)
At the start: 4 copper layers, 45 x 75 mm, 76 parts, among them J1 Conn_Coaxial, J2 Conn_ARM_JTAG_SWD_10, J3 67068-8000, J4 PLR135/T9, J5 Conn_02x07_Odd_Even, J6 Conn_01x03, U1 STM32F765NIHx, U2 MIC5355-S4YMME, U3 NBA3N012C, U4 KC3225K24.0000C1GE00, U5 USB3300-EZK, U6 ICE40HX8K-BG121, U7 KC3225K22.5792C10E00, U8 KC3225K24.5760C10E00

Commit message: First fully routed version
Parts:
- added LOGO1: Logo_Open_Hardware_Large, Symbol:OSHW-Logo2_9.8x8mm_SilkScreen, F.Cu at (161.0, 104.5)
- J5: value Conn_02x07_Odd_Even -> Conn_02x08_Odd_Even; footprint Connector_PinHeader_2.54mm:PinHeader_2x07_P2.54mm_Vertical -> Connector_PinHeader_2.54mm:PinHeader_2x08_P2.54mm_Vertical
- moved J1 3.75 mm to (146.3, 38.5)
Connections:
- J5 pad 10: /CONNECTORS/RST2 -> /CONNECTORS/RESET2
- J5 pad 13: GND -> /CONNECTORS/VDD
- J5 pad 14: GND -> /CONNECTORS/VDD
- J5 pad 9: /CONNECTORS/RST1 -> /CONNECTORS/RESET1
- U1 pad A1: Net-(U1-PadA1) -> /ICE40/CRESET
- U1 pad B1: Net-(U1-PadB1) -> /ICE40/CDONE
- U1 pad R6: Net-(U1-PadR6) -> /CONNECTORS/RESET1
- U1 pad R7: Net-(U1-PadR7) -> /CONNECTORS/RESET2
Routing:
- net /CONNECTORS/RESET1: track 0.00 -> 67.7 mm, vias 0 -> 1
- net /CONNECTORS/RESET2: track 0.00 -> 61.5 mm, vias 0 -> 1
- net /ICE40/CDONE: track 18.5 -> 55.5 mm, vias 2 -> 7
- net /ICE40/CRESET: track 4.07 -> 40.6 mm, vias 0 -> 6
- net GND: track 44.0 -> 71.4 mm, vias 54 -> 144
- net /ICE40/MOSI: track 33.8 -> 27.8 mm
- net Net-(J1-Pad1): track 8.18 -> 12.3 mm
- net /CONNECTORS/VDD5V: track 39.4 -> 42.9 mm, vias 1 -> 0
- net Net-(J1-Pad2): track 11.7 -> 15.0 mm
- net /ICE40/SCLK: track 20.7 -> 18.8 mm
- net (no net): track 1.00 -> 0.00 mm
- net /ICE40/D4: track 18.9 -> 18.3 mm, vias 2 -> 0
- net /CONNECTORS/NRST: track 20.0 -> 20.6 mm
- net /ICE40/D0: track 11.2 -> 10.8 mm, vias 2 -> 0
- net /ICE40/D7: track 15.5 -> 15.7 mm, vias 2 -> 0
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Other:
- board text added: "2019-01-12"
- board text added: "YUI"
