File: PCB/yui.sch (KiCad schematic (older format))
At the start: 0 parts

Commit message: First fully routed version
Parts:
- added LOGO1: Logo_Open_Hardware_Large, Symbol:OSHW-Logo2_9.8x8mm_SilkScreen, symbol Graphic:Logo_Open_Hardware_Large
Changed lines of the file:
@@
 F44 "SPDIF_TOSLINK" I L 7800 1400 50
 F45 "SS" I L 7800 4000 50
+F46 "CRESET" I R 9600 2450 50
+F47 "CDONE" I R 9600 2550 50
+F48 "RESET1" I L 7800 2000 50
+F49 "RESET2" I L 7800 2100 50
 $EndSheet
 $Sheet
@@
 F11 "I2S_WS_2" I R 2750 5900 50
 F12 "I2S_MCLK_2" I R 2750 6000 50
-F13 "RST1" I R 2750 2000 50
-F14 "RST2" I R 2750 2100 50
-F15 "I2C_SDA" I R 2750 1900 50
-F16 "I2C_SCL" I R 2750 1800 50
-F17 "RX" I R 2750 1700 50
-F18 "TX" I R 2750 1600 50
-F19 "NRST" I R 2750 1000 50
-F20 "SWDIO" I R 2750 1200 50
-F21 "SWDCLK" I R 2750 1100 50
-F22 "SWO" O R 2750 1300 50
-F23 "VDD" I R 2750 2250 50
-F24 "VDD3V3" I R 2750 6550 50
-F25 "SPDIF_TOSLINK" I R 2750 1400 50
-F26 "SPDIF_COAXIAL" I R 2750 1500 50
+F13 "I2C_SDA" I R 2750 1900 50
+F14 "I2C_SCL" I R 2750 1800 50
+F15 "RX" I R 2750 1700 50
+F16 "TX" I R 2750 1600 50
+F17 "NRST" I R 2750 1000 50
+F18 "SWDIO" I R 2750 1200 50
+F19 "SWDCLK" I R 2750 1100 50
+F20 "SWO" O R 2750 1300 50
+F21 "VDD" I R 2750 2250 50
+F22 "VDD3V3" I R 2750 6550 50
+F23 "SPDIF_TOSLINK" I R 2750 1400 50
+F24 "SPDIF_COAXIAL" I R 2750 1500 50
+F25 "RESET1" I R 2750 2000 50
+F26 "RESET2" I R 2750 2100 50
 $EndSheet
 Wire Wire Line
@@
 Wire Wire Line
 	7600 4900 7800 4900
+Wire Wire Line
+	7800 2000 2750 2000
+Wire Wire Line
+	2750 2100 7800 2100
+Wire Wire Line
+	10450 2550 10450 4700
+Wire Wire Line
+	10450 4700 9600 4700
+Wire Wire Line
+	9600 4600 10500 4600
+Wire Wire Line
+	10500 4600 10500 2450
+Wire Wire Line
+	10500 2450 9600 2450
+Wire Wire Line
+	9600 2550 10450 2550
+$Comp
+L Graphic:Logo_Open_Hardware_Large LOGO1
+U 1 1 5C3E8A8E
+P 6250 7150
+F 0 "LOGO1" H 6250 7650 50  0001 C CNN
+F 1 "Logo_Open_Hardware_Large" H 6250 6750 50  0001 C CNN
+F 2 "Symbol:OSHW-Logo2_9.8x8mm_SilkScreen" H 6250 7150 50  0001 C CNN
+F 3 "~" H 6250 7150 50  0001 C CNN
+	1    6250 7150
+	1    0    0    -1
+$EndComp
 $EndSCHEMATC
